File: hw/can_gauge.kicad_sch (KiCad schematic)
At the start: 21 parts, among them U1 PIC16F1459-ISS, U2 MCP2515-xSO, U3 74HC595, U4 74HC595, U5 74HC595, U6 ULN2003A, U7 ULN2003A, U8 ULN2003A

Commit message: hw: ic footprints
Parts:
- removed U2: MCP2515-xSO, Package_DIP:DIP-18_W7.62mm, symbol Interface_CAN_LIN:MCP2515-xSO
- removed XCVR1: MCP2561-E-P, Package_DIP:DIP-8_W7.62mm, symbol Interface_CAN_LIN:MCP2561-E-P
- added U10: MCP2515-xST, Package_SO:TSSOP-20_4.4x6.5mm_P0.65mm, symbol Interface_CAN_LIN:MCP2515-xST
- added U9: MCP2561T-E/SN, Package_SO:SOIC-8_3.9x4.9mm_P1.27mm, symbol Interface_CAN_LIN:MCP2561-E-SN
- U1: footprint (none) -> Package_SO:SSOP-20_5.3x7.2mm_P0.65mm
- U3, U4, U5: footprint (none) -> Package_SO:TSSOP-16_4.4x5mm_P0.65mm
- U6, U7, U8: footprint (none) -> Package_SO:SO-16_3.9x9.9mm_P1.27mm
- Vreg1: value LM2940xT -> LM2940IMPX-5.0/NOPB; footprint Package_TO_SOT_THT:TO-220-3_Vertical -> Package_TO_SOT_SMD:SOT-223
Connections:
- net +5V: now also U10.20 (VDD), U9.3 (VDD)
- net CAN_H: now also U9.7 (CANH)
- net CAN_L: now also U9.6 (CANL)
- net CLK: now also U10.9 (OSC1)
- net GND: now also U10.10 (VSS), U9.2 (VSS), U9.8 (STBY)
- net RX: now also U10.2 (RXCAN), U9.4 (RXD)
- net SCK: now also U10.14 (SCK)
- net SI: now also U10.17 (SO)
- net SO: now also U10.16 (SI)
- net TX: now also U10.1 (TXCAN), U9.1 (TXD)
- net ~{CS}: now also U10.18 (~{CS})
- net ~{INT}: now also U10.13 (~{INT})
- net at R4.1: now also U10.19 (~{RESET})
Changed lines of the file:
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@@
 			)
 		)
-		(property "Value" "LM2940xT"
+		(property "Value" "LM2940IMPX-5.0/NOPB"
 			(at 121.92 224.79 0)
 			(effects
@@
 			)
 		)
-		(property "Footprint" "Package_TO_SOT_THT:TO-220-3_Vertical"
+		(property "Footprint" "Package_TO_SOT_SMD:SOT-223"
 			(at 121.92 224.155 0)
 			(effects
@@
 			)
 		)
-		(property "Datasheet" "https://www.ti.com/lit/ds/symlink/lm2940-n.pdf?HQS=dis-dk-null-digikeymode-dsf-pf-null-wwe&ts=1748878933216&ref_url=https%253A%252F%252Fwww.ti.com%252Fgeneral%252Fdocs%252Fsuppproductinfo.tsp%253FdistId%253D10%2526gotoUrl%253Dhttps%253A%252F%252Fwww.ti.com%252Flit%252Fgpn%252Flm2940-n"
+		(property "Datasheet" "https://www.ti.com/general/docs/suppproductinfo.tsp?distId=10&gotoUrl=https%3A%2F%2Fwww.ti.com%2Flit%2Fgpn%2Flm2940-n"
 			(at 121.92 231.14 0)
 			(effects
@@
 			)
 		)
-		(property "Footprint" ""
+		(property "Footprint" "Package_SO:SSOP-20_5.3x7.2mm_P0.65mm"
 			(at 173.99 52.07 0)
 			(effects
@@
 	)
 	(symbol
+		(lib_id "Interface_CAN_LIN:MCP2515-xST")
+		(at 50.8 55.88 0)
+		(unit 1)
+		(exclude_from_sim no)
+		(in_bom yes)
+		(on_board yes)
+		(dnp no)
+		(fields_autoplaced yes)
+		(property "Reference" "U10"
+			(at 52.9433 33.02 0)
+			(effects
+				(font
+					(size 1.27 1.27)
+				)
+				(justify left)
+			)
+		)
+		(property "Value" "MCP2515-xST"
+			(at 52.9433 35.56 0)
+			(effects
+				(font
+					(size 1.27 1.27)
+				)
+				(justify left)
+			)
+		)
+		(property "Footprint" "Package_SO:TSSOP-20_4.4x6.5mm_P0.65mm"
+			(at 50.8 78.74 0)
+			(effects
+				(font
+					(size 1.27 1.27)
+					(italic yes)
+				)
+				(hide yes)
+			)
+		)
+		(property "Datasheet" "http://ww1.microchip.com/downloads/en/DeviceDoc/21801e.pdf"
+			(at 53.34 76.2 0)
+			(effects
+				(font
+					(size 1.27 1.27)
+				)
+				(hide yes)
+			)
+		)
+		(property "Description" "Stand-Alone CAN Controller with SPI Interface, TSSOP-20"
+			(at 50.8 55.88 0)
+			(effects
+				(font
+					(size 1.27 1.27)
+				)
+				(hide yes)
+			)
+		)
+		(pin "5"
+		)
+		(pin "18"
+		)
+		(pin "20"
+		)
+		(pin "19"
+		)
+		(pin "14"
+		)
+		(pin "7"
+		)
+		(pin "6"
+		)
+		(pin "10"
+		)
+		(pin "3"
+		)
+		(pin "15"
+		)
+		(pin "12"
+		)
+		(pin "1"
+		)
+		(pin "4"
+		)
+		(pin "2"
+		)
+		(pin "9"
+		)
+		(pin "11"
+		)
+		(pin "17"
+		)
+		(pin "16"
+		)
+		(pin "8"
+		)
+		(pin "13"
+		)
+		(instances
+			(project ""
+				(path "/a1545928-1195-40b9-b3c4-78f837012afb"
+					(reference "U10")
+					(unit 1)
+				)
+			)
+		)
+	)
+	(symbol
 		(lib_id "74xx:74HC595")
 		(at 267.97 128.27 0)
@@
 			)
 		)
-		(property "Footprint" ""
+		(property "Footprint" "Package_SO:TSSOP-16_4.4x5mm_P0.65mm"
 			(at 267.97 128.27 0)
 			(effects
@@
 	)
 	(symbol
+		(lib_id "Interface_CAN_LIN:MCP2561-E-SN")
+		(at 50.8 127 0)
+		(unit 1)
+		(exclude_from_sim no)
+		(in_bom yes)
+		(on_board yes)
+		(dnp no)
+		(property "Reference" "U9"
+			(at 52.9433 114.3 0)
+			(effects
+				(font
+					(size 1.27 1.27)
+				)
+				(justify left)
+			)
+		)
+		(property "Value" "MCP2561T-E/SN"
+			(at 52.9433 116.84 0)
+			(effects
+				(font
+					(size 1.27 1.27)
+				)
+				(justify left)
+			)
+		)
+		(property "Footprint" "Package_SO:SOIC-8_3.9x4.9mm_P1.27mm"
+			(at 50.8 139.7 0)
+			(effects
+				(font
+					(size 1.27 1.27)
+					(italic yes)
+				)
+				(hide yes)
+			)
+		)
+		(property "Datasheet" "https://ww1.microchip.com/downloads/en/DeviceDoc/20005167C.pdf"
+			(at 50.8 127 0)
+			(effects
+				(font
+					(size 1.27 1.27)
+				)
+				(hide yes)
+			)
+		)
+		(property "Description" "High-Speed CAN Transceiver, 1Mbps, 5V supply, SPLIT pin, -40C to +125C, SOIC-8"
+			(at 50.8 127 0)
+			(effects
+				(font
+					(size 1.27 1.27)
+				)
+				(hide yes)
+			)
+		)
+		(pin "3"
+		)
+		(pin "5"
+		)
+		(pin "7"
+		)
+		(pin "8"
+		)
+		(pin "4"
+		)
+		(pin "1"
+		)
+		(pin "6"
+		)
+		(pin "2"
+		)
+		(instances
+			(project ""
+				(path "/a1545928-1195-40b9-b3c4-78f837012afb"
+					(reference "U9")
+					(unit 1)
+				)
+			)
+		)
+	)
+	(symbol
 		(lib_id "Connector:DIN41612_02x16_AB")
 		(at 59.69 220.98 0)
@@
 	)
 	(symbol
-		(lib_id "Interface_CAN_LIN:MCP2561-E-P")
-		(at 50.8 127 0)
-		(unit 1)
-		(exclude_from_sim no)
-		(in_bom yes)
-		(on_board yes)
-		(dnp no)
-		(fields_autoplaced yes)
-		(property "Reference" "XCVR1"
-			(at 52.8194 114.3 0)
-			(effects
-				(font
-					(size 1.27 1.27)
-				)
-				(justify left)
-			)
-		)
-		(property "Value" "MCP2561-E-P"
-			(at 52.8194 116.84 0)
-			(effects
-				(font
-					(size 1.27 1.27)
-				)
-				(justify left)
-			)
-		)
-		(property "Footprint" "Package_DIP:DIP-8_W7.62mm"
-			(at 50.8 139.7 0)
-			(effects
-				(font
-					(size 1.27 1.27)
-					(italic yes)
-				)
-				(hide yes)
-			)
-		)
-		(property "Datasheet" "http://ww1.microchip.com/downloads/en/DeviceDoc/25167A.pdf"
-			(at 50.8 127 0)
-			(effects
-				(font
-					(size 1.27 1.27)
-				)
-				(hide yes)
-			)
-		)
-		(property "Description" ""
-			(at 50.8 127 0)
-			(effects
-				(font
-					(size 1.27 1.27)
-				)
-			)
-		)
-		(pin "1"
-		)
-		(pin "2"
-		)
-		(pin "3"
-		)
-		(pin "4"
-		)
-		(pin "5"
-		)
-		(pin "6"
-		)
-		(pin "7"
-		)
-		(pin "8"
-		)
-		(instances
-			(project ""
-				(path "/a1545928-1195-40b9-b3c4-78f837012afb"
-					(reference "XCVR1")
-					(unit 1)
-				)
-			)
-		)
-	)
-	(symbol
 		(lib_name "+5V_4")
 		(lib_id "power:+5V")
@@
 			)
 		)
-		(property "Footprint" ""
+		(property "Footprint" "Package_SO:SO-16_3.9x9.9mm_P1.27mm"
 			(at 332.74 134.62 0)
 			(effects
@@
 			)
 		)
-		(property "Footprint" ""
+		(property "Footprint" "Package_SO:SO-16_3.9x9.9mm_P1.27mm"
 			(at 332.74 73.66 0)
 			(effects
@@
 			)
 		)
-		(property "Footprint" ""
+		(property "Footprint" "Package_SO:SO-16_3.9x9.9mm_P1.27mm"
 			(at 332.74 195.58 0)
 			(effects
@@
 			)
 		)
-		(property "Footprint" ""
+		(property "Footprint" "Package_SO:TSSOP-16_4.4x5mm_P0.65mm"
 			(at 267.97 64.77 0)
 			(effects
@@
 			)
 		)
-		(property "Footprint" ""
+		(property "Footprint" "Package_SO:TSSOP-16_4.4x5mm_P0.65mm"
 			(at 267.97 191.77 0)
 			(effects
@@
 					(unit 1)
 				)
-			)
-		)
-	)
-	(symbol
-		(lib_id "Interface_CAN_LIN:MCP2515-xSO")
-		(at 50.8 55.88 0)
-		(unit 1)
-		(exclude_from_sim no)
-		(in_bom yes)
-		(on_board yes)
-		(dnp no)
-		(fields_autoplaced yes)
-		(property "Reference" "U2"
-			(at 52.9433 33.02 0)
-			(effects
-				(font
-					(size 1.27 1.27)
-				)
-				(justify left)
-			)
-		)
-		(property "Value" "MCP2515-xSO"
-			(at 52.9433 35.56 0)
-			(effects
-				(font
-					(size 1.27 1.27)
-				)
-				(justify left)
-			)
-		)
-		(property "Footprint" "Package_DIP:DIP-18_W7.62mm"
-			(at 50.8 78.74 0)
-			(effects
-				(font
-					(size 1.27 1.27)
-					(italic yes)
-				)
-				(hide yes)
-			)
-		)
-		(property "Datasheet" "http://ww1.microchip.com/downloads/en/DeviceDoc/21801e.pdf"
-			(at 53.34 76.2 0)
-			(effects
-				(font
-					(size 1.27 1.27)
-				)
-				(hide yes)
-			)
-		)
-		(property "Description" "Stand-Alone CAN Controller with SPI Interface, SOIC-18"
-			(at 50.8 55.88 0)
-			(effects
-				(font
-					(size 1.27 1.27)
-				)
-				(hide yes)
-			)
-		)
-		(pin "6"
-		)
-		(pin "10"
-		)
-		(pin "8"
-		)
-		(pin "2"
-		)
-		(pin "12"
-		)
-		(pin "1"
-		)
-		(pin "9"
-		)
-		(pin "3"
-		)
-		(pin "15"
-		)
-		(pin "16"
-		)
-		(pin "14"
-		)
-		(pin "13"
-		)
-		(pin "17"
-		)
-		(pin "5"
-		)
-		(pin "7"
-		)
-		(pin "18"
-		)
-		(pin "4"
-		)
-		(pin "11"
-		)
-		(instances
-			(project ""
-				(path "/a1545928-1195-40b9-b3c4-78f837012afb"
-					(reference "U2")
-					(unit 1)
-				)

Commit message: hw: rename passives
Parts:
- renumbered C8 to C1, C9 to C2, C4 to C3, C3 to C4, C1 to C5, C7 to C6, C5 to C6, R5 to R1, R4 to R2
Changed lines of the file:
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@@
 		(dnp no)
 		(fields_autoplaced yes)
-		(property "Reference" "R5"
+		(property "Reference" "R1"
 			(at 106.68 45.72 90)
 			(effects
@@
 			(project ""
 				(path "/a1545928-1195-40b9-b3c4-78f837012afb"
-					(reference "R5")
+					(reference "R1")
 					(unit 1)
 				)
@@
 		(dnp no)
 		(fields_autoplaced yes)
-		(property "Reference" "C8"
+		(property "Reference" "C1"
 			(at 107.95 231.1462 0)
 			(effects
@@
 			(project ""
 				(path "/a1545928-1195-40b9-b3c4-78f837012afb"
-					(reference "C8")
+					(reference "C1")
 					(unit 1)
 				)
@@
 		(dnp no)
 		(fields_autoplaced yes)
-		(property "Reference" "C4"
+		(property "Reference" "C3"
 			(at 180.3463 19.05 90)
 			(effects
@@
 			(project ""
 				(path "/a1545928-1195-40b9-b3c4-78f837012afb"
-					(reference "C4")
+					(reference "C3")
 					(unit 1)
 				)
@@
 		(dnp no)
 		(fields_autoplaced yes)
-		(property "Reference" "C1"
+		(property "Reference" "C5"
 			(at 57.1563 100.33 90)
 			(effects
@@
 			(project ""
 				(path "/a1545928-1195-40b9-b3c4-78f837012afb"
-					(reference "C1")
+					(reference "C5")
 					(unit 1)
 				)
@@
 		(dnp no)
 		(fields_autoplaced yes)
-		(property "Reference" "C3"
+		(property "Reference" "C4"
 			(at 57.1563 20.32 90)
 			(effects
@@
 			(project ""
 				(path "/a1545928-1195-40b9-b3c4-78f837012afb"
-					(reference "C3")
+					(reference "C4")
 					(unit 1)
 				)
@@
 		(dnp no)
 		(fields_autoplaced yes)
-		(property "Reference" "C7"
+		(property "Reference" "C6"
 			(at 274.3263 165.1 90)
 			(effects
@@
 			(project "can_gauge"
 				(path "/a1545928-1195-40b9-b3c4-78f837012afb"
-					(reference "C7")
+					(reference "C6")
 					(unit 1)
 				)
@@
 		(dnp no)
 		(fields_autoplaced yes)
-		(property "Reference" "R4"
+		(property "Reference" "R2"
 			(at 71.12 64.77 90)
 			(effects
@@
 			(project ""
 				(path "/a1545928-1195-40b9-b3c4-78f837012afb"
-					(reference "R4")
+					(reference "R2")
 					(unit 1)
 				)
@@
 		(dnp no)
 		(fields_autoplaced yes)
-		(property "Reference" "C9"
+		(property "Reference" "C2"
 			(at 134.62 230.5938 0)
 			(effects
@@
 			(project ""
 				(path "/a1545928-1195-40b9-b3c4-78f837012afb"
-					(reference "C9")
+					(reference "C2")
 					(unit 1)
 				)
@@
 		(dnp no)
 		(fields_autoplaced yes)
-		(property "Reference" "C5"
+		(property "Reference" "C6"
 			(at 274.3263 38.1 90)
 			(effects
@@
 			(project ""
 				(path "/a1545928-1195-40b9-b3c4-78f837012afb"
-					(reference "C5")
+					(reference "C6")
 					(unit 1)
 				)

Commit message: hw: passive footprints
Parts:
- added C3: 22 uF, Capacitor_Tantalum_SMD:CP_EIA-6032-28_Kemet-C, symbol Device:C_Polarized_Small
- C1: footprint Capacitor_THT:C_Disc_D5.0mm_W2.5mm_P2.50mm -> Capacitor_SMD:C_0603_1608Metric; Digikey (none) -> https://www.digikey.ca/en/products/detail/samsung-electro-m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
- C2: value 47 uF -> 22 uF; footprint (none) -> Capacitor_Tantalum_SMD:CP_EIA-6032-28_Kemet-C; Digikey (none) -> https://www.digikey.ca/en/products/detail/kyocera-avx/TAJC2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; ESR 500 m -> 1 Ohm
- C4: renamed from C3; footprint (none) -> Capacitor_SMD:C_0402_1005Metric; Digikey (none) -> https://www.digikey.ca/en/products/detail/murata-electronic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
- C5: renamed from C4; footprint (none) -> Capacitor_SMD:C_0402_1005Metric; Digikey (none) -> https://www.digikey.ca/en/products/detail/murata-electronic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
- C6: renamed from C5; footprint (none) -> Capacitor_SMD:C_0402_1005Metric; Digikey (none) -> https://www.digikey.ca/en/products/detail/murata-electronic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
- C7, C8, C9: renamed from C6; footprint (none) -> Capacitor_SMD:C_0402_1005Metric; Digikey (none) -> https://www.digikey.ca/en/products/detail/murata-electronic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
- R1, R2: footprint (none) -> Resistor_SMD:R_0402_1005Metric; Digikey (none) -> https://www.digikey.ca/en/products/detail/panasonic-electro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
Connections:
- net +5V: now also C3.1
- net GND: now also C3.2

Commit message: hw: rename ICs
Parts:
- removed J1: ~, symbol Connector:DIN41612_02x16_AB
- added J1: Gauge 1, Connector_Molex:Molex_Mini-Fit_Jr_5569-04A2_2x02_P4.20mm_Horizontal, symbol Connector_Generic:Conn_02x02_Counter_Clockwise
- added J2: Gauge 2, Connector_Molex:Molex_Mini-Fit_Jr_5569-04A2_2x02_P4.20mm_Horizontal, symbol Connector_Generic:Conn_02x02_Counter_Clockwise
- added J3: Gauge 3, Connector_Molex:Molex_Mini-Fit_Jr_5569-04A2_2x02_P4.20mm_Horizontal, symbol Connector_Generic:Conn_02x02_Counter_Clockwise
- added J4: Gauge 4, Connector_Molex:Molex_Mini-Fit_Jr_5569-04A2_2x02_P4.20mm_Horizontal, symbol Connector_Generic:Conn_02x02_Counter_Clockwise
- added J5: Gauge 5, Connector_Molex:Molex_Mini-Fit_Jr_5569-04A2_2x02_P4.20mm_Horizontal, symbol Connector_Generic:Conn_02x02_Counter_Clockwise
- added J6: Power and CAN, Connector_Molex:Molex_Mini-Fit_Jr_5569-04A2_2x02_P4.20mm_Horizontal, symbol Connector_Generic:Conn_02x02_Counter_Clockwise
- renumbered U10 to U2, U9 to U3, U3 to U4, U4 to U5, U5 to U6, U6 to U7, U7 to U8, U8 to U9
Connections:
- net +12V: now also J6.4 (Pin_4)
- net CAN_H: now also J6.1 (Pin_1)
- net CAN_L: now also J6.3 (Pin_3)
- net GND: now also J6.2 (Pin_2)
- net M1P1: now also J1.1 (Pin_1)
- net M1P2: now also J1.2 (Pin_2)
- net M1P3: now also J1.3 (Pin_3)
- net M1P4: now also J1.4 (Pin_4)
- net M2P1: now also J2.1 (Pin_1)
- net M2P2: now also J2.2 (Pin_2)
- net M2P3: now also J2.3 (Pin_3)
- net M2P4: now also J2.4 (Pin_4)
- net M3P1: now also J3.1 (Pin_1)
- net M3P2: now also J3.2 (Pin_2)
- net M3P3: now also J3.3 (Pin_3)
- net M3P4: now also J3.4 (Pin_4)
- net M4P1: now also J4.1 (Pin_1)
- net M4P2: now also J4.2 (Pin_2)
- net M4P3: now also J4.3 (Pin_3)
- net M4P4: now also J4.4 (Pin_4)
- net M5P1: now also J5.1 (Pin_1)
- net M5P2: now also J5.2 (Pin_2)
- net M5P3: now also J5.3 (Pin_3)
- net M5P4: now also J5.4 (Pin_4)
Other:
- moved on the sheet: C1, C2, C3, Vreg1
